Commit message: Fix critical IK safety bugs, add roll-freedom recovery, RViz diagnostics, LiDAR LPF
- piper_controller_node: fix solve_ik() joint-index off-by-one (joint6 was
  never reset, causing nondeterministic IK), reject unverified/out-of-limit
  IK solutions instead of executing them, add canonical_reach seed for large
  jumps, add roll-sweep recovery to exploit the free rotation DOF around the
  approach axis when the direct orientation request has no IK solution.
- push_forward_node: add LEVEL alignment stage docs, ENABLE_PUSH flag to test
  alignment without pushing, roll-agnostic arrival check to match the
  controller's new roll-freedom behavior, loosen arrival tolerances to match
  measured MIT PD tracking residual.
- contact_planner_node: add RViz diagnostic markers (plane normal, tip axis,
  perpendicular, plane quad, LOCK error text), raise ALIGN_STANDOFF_M 3cm->6cm
  after observing IK failures/divergence near the too-aggressive 3cm value.
- lidar_pointcloud_correction: add per-pixel temporal LPF (lpf_alpha).
- piper_with_lidar.urdf: swap lidar_1/lidar_2 joint values (mounts were
  physically swapped), retune dx corrections.
- Document today's session, open issues, and next-session candidates in
  CLAUDE.md.

Co-Authored-By: Claude Sonnet 5 <noreply@anthropic.com>

File: src/piper_description/urdf/piper_with_lidar.urdf (robot description, URDF)
Before this commit: robot piper_with_lidar, 20 links, 19 joints
Links:
- link lidar_1_link: geometry visual box size=0.024 0.037 0.037
- link lidar_2_link: geometry visual box size=0.024 0.037 0.037
Joints:
- joint extension_plate_joint: origin xyz=0.146037 0.034253 0.005 rpy=0 0 1.80118 -> xyz=0.145917 0.034763 0.005 rpy=0 0 1.804670
- joint extension_wall_left_joint: origin xyz=0.179148 -0.106916 0.03 rpy=0 0 1.80118 -> xyz=0.179520 -0.106290 0.03 rpy=0 0 1.804670
- joint extension_wall_right_joint: origin xyz=0.112926 0.175422 0.03 rpy=0 0 1.80118 -> xyz=0.112313 0.175815 0.03 rpy=0 0 1.804670
- joint lidar_1_joint: origin xyz=-0.255078 -0.0598279 0.03 rpy=0.0 -1.570796 0.230383 -> xyz=0.254867 0.060719 0.025 rpy=-1.570796 -1.570796 -1.336923
- joint lidar_1_optical_joint: origin xyz=0 0 0 rpy=0 0 0 -> xyz=0.012 0 0.0025 rpy=0 0 0
- joint lidar_2_joint: origin xyz=0.255078 0.0598279 0.03 rpy=-1.570796 -1.570796 -1.340413 -> xyz=-0.254867 -0.060719 0.025 rpy=0.0 -1.570796 0.233873
- joint lidar_2_optical_joint: origin xyz=0 0 0 rpy=0 0 0 -> xyz=0.012 0 0.0025 rpy=0 0 0
- joint mount_plate_joint: origin xyz=-0.0973579 -0.0228351 0.005 rpy=0 0 1.80118 -> xyz=-0.097278 -0.023175 0.005 rpy=0 0 1.804670
- joint wall_bottom_joint: origin xyz=0.238527 0.055946 0.03 rpy=0 0 1.80118 -> xyz=0.238330 0.056778 0.03 rpy=0 0 1.804670
- joint wall_left_joint: origin xyz=-0.064247 -0.164004 0.03 rpy=0 0 1.80118 -> xyz=-0.063674 -0.164228 0.03 rpy=0 0 1.804670
- joint wall_right_joint: origin xyz=-0.130469 0.118334 0.03 rpy=0 0 1.80118 -> xyz=-0.130882 0.117877 0.03 rpy=0 0 1.804670
- joint wall_top_joint: origin xyz=-0.238527 -0.055946 0.03 rpy=0 0 1.80118 -> xyz=-0.238330 -0.056778 0.03 rpy=0 0 1.804670
